Commit message: Improved robot model

File: ros_packages/robot_description/urdf/cortex.xacro (robot description, xacro)
@@ -12,5 +12,5 @@
     <xacro:property name="wheel_radius" value="0.03" />
     <xacro:property name="wheel_width" value="0.04" />
-    <link name="base">
+    <link name="base_link">
         <visual>
             <geometry>
@@ -23,4 +23,20 @@
         </visual>
     </link>
+    <link name="top">
+        <visual>
+            <geometry>
+                <box size="${base_length} ${base_width - 0.002} ${top_height}"/>
+            </geometry>
+            <origin rpy="0 0 0" xyz="0 0 ${base_height + base_ground_offset + top_height/2}"/>
+            <material name="pink">
+                <color rgba="1 0.7 0.7 1"/>
+            </material>
+        </visual>
+    </link>
+    <joint name="base_link_to_top" type="fixed">
+        <parent link="base_link"/>
+        <child link="top"/>
+        <origin xyz="0 0 0"/>
+    </joint>
     <xacro:macro name="wheel" params="suffix offset_x offset_y">
         <link name="wheel_${suffix}">
@@ -35,6 +51,6 @@
             </visual>
         </link>
-        <joint name="base_to_wheel_${suffix}" type="fixed">
-            <parent link="base"/>
+        <joint name="base_link_to_wheel_${suffix}" type="fixed">
+            <parent link="base_link"/>
             <child link="wheel_${suffix}"/>
             <origin xyz="0 0 0"/>

Commit message: Update robot model with physical info for simulation

File: ros_packages/robot_description/urdf/cortex.xacro (robot description, xacro)
@@ -2,35 +2,84 @@
 <robot xmlns:xacro="http://www.ros.org/wiki/xacro" name="Cortex">
     <!-- Constants -->
+    <!-- All physical properties use the metric system -->
     <xacro:property name="PI" value="3.1415926535897931" />
     <!-- Base -->
-    <xacro:property name="base_width" value="0.2" />
-    <xacro:property name="base_length" value="0.15" />
-    <xacro:property name="base_height" value="0.06" />
+    <xacro:property name="base_size_x" value="0.2" />
+    <xacro:property name="base_size_y" value="0.15" />
+    <xacro:property name="base_size_z" value="0.06" />
     <xacro:property name="base_ground_offset" value="0.01" />
-    <xacro:property name="top_height" value="0.2" />
+    <xacro:property name="base_mass" value="1" />
+    <!-- Top -->
+    <xacro:property name="top_size_z" value="0.2" />
+    <xacro:property name="top_mass" value="2" />
     <!-- Wheels -->
     <xacro:property name="wheel_radius" value="0.03" />
     <xacro:property name="wheel_width" value="0.04" />
+    <xacro:property name="wheel_mass" value="0.086" />
+    <!-- Motors -->
+    <!-- Polulu motor:  https://www.pololu.com/product/2824/specs -->
+    <!-- Max torque: 170 oz·in = 1.2 Nm -->
+    <xacro:property name="motor_max_torque" value="1.2" />
+    <!-- Max velocity: 200 rpm = 20 rad/s -->
+    <xacro:property name="motor_max_velocity" value="20" />
+    <!-- Macros for inertia -->
+    <xacro:macro name="default_inertial" params="mass">
+        <inertial>
+            <mass value="${mass}" />
+            <inertia ixx="1.0" ixy="0.0" ixz="0.0"
+                     iyy="1.0" iyz="0.0"
+                     izz="1.0" />
+        </inertial>
+    </xacro:macro>
+    <xacro:macro name="box_inertial" params="mass x y z">
+        <inertial>
+            <mass value="${mass}" />
+            <inertia ixx="${1/12 * mass * (z**2 + y**2)}" ixy="0.0" ixz="0.0"
+                     iyy="${1/12 * mass * (x**2 + y**2)}" iyz="0.0"
+                     izz="${1/12 * mass * (x**2 + z**2)}" />
+        </inertial>
+    </xacro:macro>
+    <xacro:macro name="cylinder_inertial" params="mass r z">
+        <inertial>
+            <mass value="${mass}" />
+            <inertia ixx="${1/12 * mass * (3 * r**2 + z**2)}" ixy="0.0" ixz="0.0"
+                     iyy="${1/12 * mass * (3 * r**2 + z**2)}" iyz="0.0"
+                     izz="${1/2 * mass * r**2}" />
+        </inertial>
+    </xacro:macro>
+    <!-- Links -->
     <link name="base_link">
         <visual>
             <geometry>
-                <box size="${base_length} ${base_width - 0.002} ${base_height}"/>
+                <box size="${base_size_x - 0.002} ${base_size_y} ${base_size_z}"/>
             </geometry>
-            <origin rpy="0 0 0" xyz="0 0 ${base_height/2 + base_ground_offset}"/>
+            <origin rpy="0 0 0" xyz="0 0 ${base_size_z/2 + base_ground_offset}"/>
             <material name="white">
                 <color rgba="1 1 1 1"/>
             </material>
         </visual>
+        <collision>
+            <geometry>
+                <box size="${base_size_x - 0.002} ${base_size_y} ${base_size_z}"/>
+            </geometry>
+        </collision>
+        <xacro:box_inertial mass="${base_mass}" x="${base_size_x}" y="${base_size_y}" z="${base_size_z}"/>
     </link>
     <link name="top">
         <visual>
             <geometry>
-                <box size="${base_length} ${base_width - 0.002} ${top_height}"/>
+                <box size="${base_size_x - 0.002} ${base_size_y} ${top_size_z}"/>
             </geometry>
-            <origin rpy="0 0 0" xyz="0 0 ${base_height + base_ground_offset + top_height/2}"/>
+            <origin rpy="0 0 0" xyz="0 0 ${base_size_z + base_ground_offset + top_size_z/2}"/>
             <material name="pink">
                 <color rgba="1 0.7 0.7 1"/>
             </material>
         </visual>
+        <collision>
+            <geometry>
+                <box size="${base_size_x - 0.002} ${base_size_y} ${top_size_z}"/>
+            </geometry>
+        </collision>
+        <xacro:box_inertial mass="${top_mass}" x="${base_size_x}" y="${base_size_y}" z="${top_size_z}"/>
     </link>
     <joint name="base_link_to_top" type="fixed">
@@ -45,19 +94,22 @@
                     <cylinder length="${wheel_width}" radius="${wheel_radius}"/>
                 </geometry>
-                <origin rpy="${PI/2} 0 0" xyz="${offset_x} ${offset_y} ${wheel_radius}"/>
+                <origin rpy="0 ${PI/2} 0" /> <!-- xyz="${offset_x} ${offset_y} ${wheel_radius}" -->
                 <material name="black">
                     <color rgba="0 0 0 1"/>
                 </material>
             </visual>
+            <xacro:cylinder_inertial mass="${wheel_mass}" r="${wheel_radius}" z="${wheel_width}"/>
         </link>
-        <joint name="base_link_to_wheel_${suffix}" type="fixed">
+        <joint name="base_link_to_wheel_${suffix}" type="continuous">
             <parent link="base_link"/>
             <child link="wheel_${suffix}"/>
-            <origin xyz="0 0 0"/>
+            <axis xyz="1 0 0"/>
+            <origin xyz="${offset_x} ${offset_y} ${wheel_radius}"/>
+            <limit effort ="${motor_max_torque}" velocity="${motor_max_velocity}"/>
         </joint>
     </xacro:macro>
-    <xacro:wheel suffix="front_left" offset_x="${base_length/2 - wheel_radius}" offset_y="${-(base_width/2 - wheel_width/2)}"/>
-    <xacro:wheel suffix="front_right" offset_x="${base_length/2 - wheel_radius}" offset_y="${base_width/2 - wheel_width/2}"/>
-    <xacro:wheel suffix="rear_left" offset_x="${-(base_length/2 - wheel_radius)}" offset_y="${-(base_width/2 - wheel_width/2)}"/>
-    <xacro:wheel suffix="rear_right" offset_x="${-(base_length/2 - wheel_radius)}" offset_y="${base_width/2 - wheel_width/2}"/>
+    <xacro:wheel suffix="front_left" offset_y="${base_size_y/2 - wheel_radius}" offset_x="${-(base_size_x/2 - wheel_width/2)}"/>
+    <xacro:wheel suffix="front_right" offset_y="${base_size_y/2 - wheel_radius}" offset_x="${base_size_x/2 - wheel_width/2}"/>
+    <xacro:wheel suffix="rear_left" offset_y="${-(base_size_y/2 - wheel_radius)}" offset_x="${-(base_size_x/2 - wheel_width/2)}"/>
+    <xacro:wheel suffix="rear_right" offset_y="${-(base_size_y/2 - wheel_radius)}" offset_x="${base_size_x/2 - wheel_width/2}"/>
 </robot>

Commit message: Macanum encoder feedback to odometry

File: ros_packages/robot_description/urdf/cortex.xacro (robot description, xacro)
@@ -5,11 +5,11 @@
     <xacro:property name="PI" value="3.1415926535897931" />
     <!-- Base -->
-    <xacro:property name="base_size_x" value="0.2" />
-    <xacro:property name="base_size_y" value="0.15" />
-    <xacro:property name="base_size_z" value="0.06" />
+    <xacro:property name="base_size_width" value="0.2" />
+    <xacro:property name="base_size_length" value="0.15" />
+    <xacro:property name="base_size_height" value="0.06" />
     <xacro:property name="base_ground_offset" value="0.01" />
     <xacro:property name="base_mass" value="1" />
     <!-- Top -->
-    <xacro:property name="top_size_z" value="0.2" />
+    <xacro:property name="top_size_height" value="0.2" />
     <xacro:property name="top_mass" value="2" />
     <!-- Wheels -->
@@ -52,7 +52,7 @@
         <visual>
             <geometry>
-                <box size="${base_size_x - 0.002} ${base_size_y} ${base_size_z}"/>
+                <box size="${base_size_length} ${base_size_width - 0.002} ${base_size_height}"/>
             </geometry>
-            <origin rpy="0 0 0" xyz="0 0 ${base_size_z/2 + base_ground_offset}"/>
+            <origin rpy="0 0 0" xyz="0 0 ${base_size_height/2 + base_ground_offset}"/>
             <material name="white">
                 <color rgba="1 1 1 1"/>
@@ -61,15 +61,15 @@
         <collision>
             <geometry>
-                <box size="${base_size_x - 0.002} ${base_size_y} ${base_size_z}"/>
+                <box size="${base_size_length} ${base_size_width - 0.002} ${base_size_height}"/>
             </geometry>
         </collision>
-        <xacro:box_inertial mass="${base_mass}" x="${base_size_x}" y="${base_size_y}" z="${base_size_z}"/>
+        <xacro:box_inertial mass="${base_mass}" x="${base_size_length}" y="${base_size_width}" z="${base_size_height}"/>
     </link>
     <link name="top">
         <visual>
             <geometry>
-                <box size="${base_size_x - 0.002} ${base_size_y} ${top_size_z}"/>
+                <box size="${base_size_length} ${base_size_width - 0.002} ${top_size_height}"/>
             </geometry>
-            <origin rpy="0 0 0" xyz="0 0 ${base_size_z + base_ground_offset + top_size_z/2}"/>
+            <origin rpy="0 0 0" xyz="0 0 ${base_size_height + base_ground_offset + top_size_height/2}"/>
             <material name="pink">
                 <color rgba="1 0.7 0.7 1"/>
@@ -78,8 +78,8 @@
         <collision>
             <geometry>
-                <box size="${base_size_x - 0.002} ${base_size_y} ${top_size_z}"/>
+                <box size="${base_size_length} ${base_size_width - 0.002} ${top_size_height}"/>
             </geometry>
         </collision>
-        <xacro:box_inertial mass="${top_mass}" x="${base_size_x}" y="${base_size_y}" z="${top_size_z}"/>
+        <xacro:box_inertial mass="${top_mass}" x="${base_size_length}" y="${base_size_width}" z="${top_size_height}"/>
     </link>
     <joint name="base_link_to_top" type="fixed">
@@ -94,5 +94,5 @@
                     <cylinder length="${wheel_width}" radius="${wheel_radius}"/>
                 </geometry>
-                <origin rpy="0 ${PI/2} 0" /> <!-- xyz="${offset_x} ${offset_y} ${wheel_radius}" -->
+                <origin rpy="${PI/2} 0 0" /> <!-- xyz="${offset_x} ${offset_y} ${wheel_radius}" -->
                 <material name="black">
                     <color rgba="0 0 0 1"/>
@@ -104,12 +104,12 @@
             <parent link="base_link"/>
             <child link="wheel_${suffix}"/>
-            <axis xyz="1 0 0"/>
+            <axis xyz="0 1 0"/>
             <origin xyz="${offset_x} ${offset_y} ${wheel_radius}"/>
             <limit effort ="${motor_max_torque}" velocity="${motor_max_velocity}"/>
         </joint>
     </xacro:macro>
-    <xacro:wheel suffix="front_left" offset_y="${base_size_y/2 - wheel_radius}" offset_x="${-(base_size_x/2 - wheel_width/2)}"/>
-    <xacro:wheel suffix="front_right" offset_y="${base_size_y/2 - wheel_radius}" offset_x="${base_size_x/2 - wheel_width/2}"/>
-    <xacro:wheel suffix="rear_left" offset_y="${-(base_size_y/2 - wheel_radius)}" offset_x="${-(base_size_x/2 - wheel_width/2)}"/>
-    <xacro:wheel suffix="rear_right" offset_y="${-(base_size_y/2 - wheel_radius)}" offset_x="${base_size_x/2 - wheel_width/2}"/>
+    <xacro:wheel suffix="front_left" offset_x="${base_size_length/2 - wheel_radius}" offset_y="${-(base_size_width/2 - wheel_width/2)}"/>
+    <xacro:wheel suffix="front_right" offset_x="${base_size_length/2 - wheel_radius}" offset_y="${base_size_width/2 - wheel_width/2}"/>
+    <xacro:wheel suffix="rear_left" offset_x="${-(base_size_length/2 - wheel_radius)}" offset_y="${-(base_size_width/2 - wheel_width/2)}"/>
+    <xacro:wheel suffix="rear_right" offset_x="${-(base_size_length/2 - wheel_radius)}" offset_y="${base_size_width/2 - wheel_width/2}"/>
 </robot>

Commit message: Begin strategy and tweak planners and costmaps for navigation

File: ros_packages/robot_description/urdf/cortex.xacro (robot description, xacro)
@@ -5,6 +5,6 @@
     <xacro:property name="PI" value="3.1415926535897931" />
     <!-- Base -->
-    <xacro:property name="base_size_width" value="0.2" />
-    <xacro:property name="base_size_length" value="0.15" />
+    <xacro:property name="base_size_width" value="0.25" />
+    <xacro:property name="base_size_length" value="0.16" />
     <xacro:property name="base_size_height" value="0.06" />
     <xacro:property name="base_ground_offset" value="0.01" />

Commit message: Ultrasound in model

File: ros_packages/robot_description/urdf/cortex.xacro (robot description, xacro)
@@ -17,4 +17,8 @@
     <xacro:property name="wheel_width" value="0.04" />
     <xacro:property name="wheel_mass" value="0.086" />
+    <xacro:property name="wheel_mass" value="0.086" />
+	<!--ultrasound -->
+	<xacro:property name="ultrasound_size_front_rear" value = "0.02 0.04 0.01" />
+    <xacro:property name="ultrasound_size_right_left" value = "0.04 0.02 0.01" />
     <!-- Motors -->
     <!-- Polulu motor:  https://www.pololu.com/product/2824/specs -->
@@ -88,4 +92,22 @@
         <origin xyz="0 0 0"/>
     </joint>
+	 <!--
+	<link name="ultrasound_rear">
+    <visual>
+      <geometry>
+        <box size="0.04 0.02 0.01"/>
+      </geometry>
+      <origin rpy="1.57079632679 0 0" xyz="-0.070 0.08 0.03"/>
+      <material name="Green">
+        <color rgba="0 1 0 1"/>
+      </material>
+    </visual>
+  </link>
+  <joint name="base_to_ultrasound_rear" type="fixed">
+    <parent link="base_link"/>
+    <child link="ultrasound_rear"/>
+    <origin xyz="0 0 0"/>
+  </joint>
+ -->
     <xacro:macro name="wheel" params="suffix offset_x offset_y">
         <link name="wheel_${suffix}">
@@ -109,7 +131,29 @@
         </joint>
     </xacro:macro>
+	<xacro:macro name="ultrasound" params="suffix offset_x offset_y offset_z rot_x rot_y rot_z">
+        <link name="ultrasound_${suffix}">
+            <visual>
+                <geometry>
+                    <box size="0.02 0.04 0.01" />
+                </geometry>
+                <origin rpy="0 0 0" xyz="0 0 0" />
+                <material name="green">
+                    <color rgba="0 1 0 1"/>
+                </material>
+            </visual>
+        </link>
+        <joint name="base_link_to_ultrasound_${suffix}" type="fixed">
+            <parent link="base_link"/>
+            <child link="ultrasound_${suffix}"/>
+           <origin rpy="${rot_x} ${rot_y} ${rot_z}" xyz="${offset_x} ${offset_y} ${offset_z}"/>
+        </joint>
+    </xacro:macro>
     <xacro:wheel suffix="front_left" offset_x="${base_size_length/2 - wheel_radius}" offset_y="${-(base_size_width/2 - wheel_width/2)}"/>
     <xacro:wheel suffix="front_right" offset_x="${base_size_length/2 - wheel_radius}" offset_y="${base_size_width/2 - wheel_width/2}"/>
     <xacro:wheel suffix="rear_left" offset_x="${-(base_size_length/2 - wheel_radius)}" offset_y="${-(base_size_width/2 - wheel_width/2)}"/>
     <xacro:wheel suffix="rear_right" offset_x="${-(base_size_length/2 - wheel_radius)}" offset_y="${base_size_width/2 - wheel_width/2}"/>
+	<xacro:ultrasound suffix="front" offset_x="${base_size_length/2 - 0.02/2}" offset_y="0" offset_z="0.03" rot_x="0" rot_y="0" rot_z="0" />
+	<xacro:ultrasound suffix="rear" offset_x="${-(base_size_length/2 - 0.02/2)}" offset_y="0" offset_z="0.03" rot_x="0" rot_y="0" rot_z="${PI}" />
+	<xacro:ultrasound suffix="left" offset_x="0" offset_y="${base_size_width/2 - 0.02/2}" offset_z="0.03" rot_x="0" rot_y="0" rot_z="${PI/2}" />
+	<xacro:ultrasound suffix="right" offset_x="0" offset_y="${-(base_size_width/2 - 0.02/2)}" offset_z="0.03" rot_x="0" rot_y="0" rot_z="${-PI/2}" />
 </robot>
